File: pcb/esphome-dot-debug.kicad_pcb (KiCad board)
At the start: 4 copper layers, 99 x 41.5 mm, 28 parts, among them J1 I2S1, J2 Conn_01x07_Pin, J3 USBC, J4 Input, SW1 PROG, U1 ESP32-S3-WROOM-2

Commit message: pcb-v1
Parts:
- moved TP2 2.06 mm to (131.6, 66.2)
- moved TP3 2.06 mm to (137.1, 66.2)
Routing:
- net ~{SPECIAL_BUTTON}: track 70.4 -> 68.6 mm
- net ~{BUTTON_INT}: track 69.5 -> 67.7 mm
Other:
- board text added: "<<hash>>"
- board text added: "GND I2S1_FS I2S1_CLK I2S1_SD 3V3"
- board text added: "GPIO14 GPIO10 GPIO17 GPIO18 GPIO46 GPIO38 GND"
- board text added: "esphome-dot-debug v1"
